File: EAGLE/Battery Shield.brd (EAGLE design)
At the start: 100 x 81.3 mm, 31 parts, among them IC1 MCP73871, U1 TPS61200

Commit message: v1.2
Parts:
- moved R7 27.7 mm to (24.7, 2.32)
- moved R8 26.8 mm to (24.9, 0.80)
- moved R9 20.3 mm to (18.9, 3.51)
- moved R10 16.5 mm to (23.5, 3.76)
- moved RT1 15.6 mm to (23.5, 4.95)
- moved C1 14.7 mm to (27.9, 2.03)
- moved C3 8.42 mm to (19.1, 7.37), turned to 90 degrees
- moved CHARGE+ 7.88 mm to (4.06, 1.52)
- moved PHONE+ 7.62 mm to (1.27, 8.89)
- moved IC1 6.15 mm to (12.1, 2.79), turned to 90 degrees
- moved C6 6.12 mm to (7.87, 3.05), turned to 270 degrees
- moved C4 6.12 mm to (4.32, 8.64), turned to 270 degrees
- moved U1 5.34 mm to (8.51, 7.87), turned to 180 degrees
- moved L1 4.71 mm to (12.3, 7.75)
- moved CHARGE- 3.61 mm to (4.06, 4.06)
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Routing:
- net GND: track 12.6 -> 3.61 mm
- net VBATT_OUT: track 6.72 -> 0.00 mm, vias 2 -> 0
- net VBUS: track 6.06 -> 0.00 mm
- net +5V: track 8.96 -> 3.22 mm
- added copper zone on layer 1, net GND
Other:
- board size 100 x 81.3 mm -> 100 x 80 mm
