File: EAGLE/Battery Shield.sch (EAGLE design)
At the start: 31 parts, among them IC1 MCP73871, U1 TPS61200

Commit message: v1.2
Other:
- note removed: "- 1"
- note removed: "Battery Shield design by Spark Devices Component libraries by Adafruit and Sparkfun"
- note removed: "R1 ="
- note removed: "R2"
- note removed: "Reference Designs ARE PROVIDED "AS IS" AND "WITH ALL FAULTS. SPARK LABS, INC ("SPARK") DISCLAIMS ALL OTHER WARRANTIES, EXPRESS OR IMPLIED, REGARDING PRODUCTS OR THE REFERENCE DESIGNS, INCLUDING BUT NOT LIMITED TO, ANY IMPLIED WARRANTIES OF MERCHANTABILITY, FITNESS FOR A PARTICULAR PURPOSE, OR NON-INFRINGEMENT. Spark may make changes to specifications and product descriptions at any time, without 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"
- note removed: "VFB"
- note removed: "Vout"
- note removed: "charge current = 1000V/PROG1"
- note removed: "recalculte RT1 and RT2 depending on the characteristics of the 10K NTC thermistor"
- note removed: "x"
Changed lines of the file:
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@@
 <layer number="96" name="Values" color="7" fill="1" visible="yes" active="yes"/>
 <layer number="97" name="Info" color="7" fill="1" visible="yes" active="yes"/>
-<layer number="98" name="Guide" color="6" fill="1" visible="yes" active="yes"/>
+<layer number="98" name="Guide" color="6" fill="1" visible="no" active="yes"/>
 <layer number="100" name="Muster" color="7" fill="1" visible="no" active="no"/>
 <layer number="101" name="Patch_Top" color="12" fill="4" visible="yes" active="yes"/>
 <layer number="102" name="Vscore" color="7" fill="1" visible="yes" active="yes"/>
 <layer number="103" name="fp3" color="7" fill="1" visible="no" active="yes"/>
-<layer number="104" name="Name" color="7" fill="1" visible="yes" active="yes"/>
+<layer number="104" name="Name" color="7" fill="1" visible="no" active="yes"/>
 <layer number="105" name="Beschreib" color="9" fill="1" visible="yes" active="yes"/>
 <layer number="106" name="BGA-Top" color="4" fill="1" visible="yes" active="yes"/>
@@
 <text x="71.12" y="63.5" size="1.778" layer="95" align="center">Battery Charger</text>
 <text x="180.34" y="63.5" size="1.778" layer="95" align="center">Boost Regulator</text>
-<text x="124.46" y="76.2" size="1.27" layer="95">recalculte RT1 and RT2
-depending on the characteristics
-of the 10K NTC thermistor</text>
-<wire x1="121.92" y1="73.66" x2="121.92" y2="83.82" width="0" layer="95"/>
-<wire x1="121.92" y1="83.82" x2="152.4" y2="83.82" width="0" layer="95"/>
-<wire x1="152.4" y1="83.82" x2="152.4" y2="73.66" width="0" layer="95"/>
-<wire x1="152.4" y1="73.66" x2="121.92" y2="73.66" width="0" layer="95"/>
-<text x="30.48" y="71.12" size="1.27" layer="95">charge current = 1000V/PROG1</text>
-<text x="214.884" y="86.106" size="1.27" layer="95">R1 = </text>
-<text x="219.456" y="86.106" size="1.27" layer="95">R2</text>
-<text x="222.25" y="86.106" size="1.27" layer="95">x</text>
-<text x="224.028" y="86.868" size="1.27" layer="95">Vout</text>
-<text x="224.282" y="84.582" size="1.27" layer="95">VFB</text>
-<text x="228.854" y="86.106" size="1.27" layer="95">- 1</text>
-<wire x1="223.774" y1="86.36" x2="228.092" y2="86.36" width="0.2032" layer="95"/>
-<wire x1="223.774" y1="88.646" x2="223.266" y2="88.138" width="0.0508" layer="95"/>
-<wire x1="223.266" y1="88.138" x2="223.266" y2="84.582" width="0.0508" layer="95"/>
-<wire x1="223.266" y1="84.582" x2="223.774" y2="84.074" width="0.0508" layer="95"/>
-<wire x1="230.886" y1="88.646" x2="231.394" y2="88.138" width="0.0508" layer="95"/>
-<wire x1="231.394" y1="88.138" x2="231.394" y2="84.582" width="0.0508" layer="95"/>
-<wire x1="231.394" y1="84.582" x2="230.886" y2="84.074" width="0.0508" layer="95"/>
-<wire x1="213.36" y1="83.82" x2="213.36" y2="88.9" width="0.0508" layer="95"/>
-<wire x1="213.36" y1="88.9" x2="233.68" y2="88.9" width="0.0508" layer="95"/>
-<wire x1="233.68" y1="88.9" x2="233.68" y2="83.82" width="0.0508" layer="95"/>
-<wire x1="233.68" y1="83.82" x2="213.36" y2="83.82" width="0.0508" layer="95"/>
 <text x="149.86" y="25.4" size="6.4516" layer="94">Spark Devices</text>
-<text x="147.32" y="36.83" size="1.27" layer="95" font="vector">Battery Shield design by Spark Devices
-Component libraries by Adafruit and Sparkfun</text>
-<text x="5.08" y="5.08" size="1.778" layer="95" font="vector">Reference Designs ARE PROVIDED "AS IS" AND "WITH ALL FAULTS. SPARK LABS, INC
-("SPARK") DISCLAIMS ALL OTHER WARRANTIES, EXPRESS OR IMPLIED, REGARDING
-PRODUCTS OR THE REFERENCE DESIGNS, INCLUDING BUT NOT LIMITED TO, ANY
-IMPLIED WARRANTIES OF MERCHANTABILITY, FITNESS FOR A PARTICULAR PURPOSE,
-OR NON-INFRINGEMENT.
-Spark may make changes to specifications and product descriptions at any
-time, without notice. The Customer must not rely on the absence or
-characteristics of any features or instructions marked "reserved" or
-"undefined." Spark reserves these for future definition and shall have
-no responsibility whatsoever for conflicts or incompatibilities arising
-from future changes to them. The product information on the Web Site or
-Materials is subject to change without notice. Do not finalize a design
-with this information.
-Spark is a registered trademark.</text>
 <text x="236.22" y="7.62" size="2.54" layer="94" font="vector">2.0.1</text>
 </plain>
@@
 <pinref part="BATT-" gate="G$1" pin="P"/>
 <wire x1="102.87" y1="106.68" x2="106.68" y2="106.68" width="0.1524" layer="91"/>
+<junction x="102.87" y="101.6"/>
 </segment>
 <segment>
@@
 <pinref part="C6" gate="G$1" pin="+"/>
 <wire x1="44.45" y1="106.68" x2="44.45" y2="109.22" width="0.1524" layer="91"/>
+<junction x="44.45" y="106.68"/>
 </segment>
 </net>
@@
 </sheet>
 </sheets>
+<errors>
+</errors>
 </schematic>
 </drawing>
-<compatibility>
-<note version="6.3" minversion="6.2.2" severity="warning">
-Since Version 6.2.2 text objects can contain more than one line,
-which will not be processed correctly with this version.
-</note>
-</compatibility>
 </eagle>
